File: elec/SHERPENT20250113/_autosave-SHERPENT20250113.kicad_sch (KiCad schematic)
At the start: 79 parts, among them J1 2137160001, Q1 NMOS, Q2 PMOS, SW1 SW_Push, U1 AN034_ANTENNA, U2 MCP73831T-2ACI_OT, U3 TPS61288LRQQR, U4 TPS7A2633DRVR, U5 LM66200DRLR, U6 ESP32-C3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

Commit message: oui
Parts:
- added D10, D11, D4, D5, D6, D7, D8, D9: WS2812B, LED_SMD:LED_WS2812B_PLCC4_5.0x5.0mm_P3.2mm, symbol LED:WS2812B
