File: elec/SHERPENT20250113/SHERPENT20250113.kicad_sch (KiCad schematic)
At the start: 134 parts, among them J1 2137160001, J2 Conn_01x03_Socket, J3 Conn_01x03_Socket, Q1 NMOS, Q2 PMOS, Q3 NMOS, Q4 PMOS, SW1 CT1102, SW2 SW_Push, U1 MCP73831T-2ACI_OT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

Commit message: Pascal was here
Parts:
- removed D4: D_Schottky, LED_SMD:LED_0603_1608Metric_Pad1.05x0.95mm_HandSolder, symbol Device:D_Schottky
- removed F1: 10A, Fuse:Fuse_0603_1608Metric, symbol Device:Fuse
- removed R18, R19: 0, Resistor_SMD:R_0603_1608Metric, symbol Device:R_US
- removed U4: LD1117S50TR_SOT223, Package_TO_SOT_SMD:SOT-223-3_TabPin2, symbol Regulator_Linear:LD1117S50TR_SOT223
- added C14, C21: 100n, Capacitor_SMD:C_0603_1608Metric_Pad1.08x0.95mm_HandSolder, symbol Device:C
- added C29: 1u, Capacitor_SMD:C_0603_1608Metric_Pad1.08x0.95mm_HandSolder, symbol Device:C
- added D26, D27: BAV99, Package_TO_SOT_SMD:SOT-23, symbol Diode:BAV99
- added D28, D4: D_Zener, Resistor_SMD:R_0603_1608Metric_Pad0.98x0.95mm_HandSolder, symbol Device:D_Zener
- added F2, F3: 10A, Fuse:Fuse_0603_1608Metric, symbol Device:Fuse
- added TP8: GND, TestPoint:TestPoint_Loop_D2.54mm_Drill1.5mm_Beaded, symbol Connector:TestPoint
- C26: value 10nf -> 10n
- R26: now not fitted
- R27: value 27.3k 0.1% -> 27.3k 1%
- R28: value 100k 0.1% -> 100k 1%
- TP1: value TestPoint -> VBATT
- TP3: value TestPoint -> USB_P
- TP5: value TestPoint -> USB_N
- TP6: value TestPoint -> GND
Connections:
- net +3.3V: now also D4.1 (K)
- net +9V: now also C29.1
- net GND: now also C14.2, C21.1, C29.2, D26.1 (K), D27.1 (K), D28.2 (A), D4.2 (A), TP8.1
- net USB_ESP32N: now also D26.3 (K)
- net USB_ESP32P: now also D27.3 (K)
- net VBATT: now also F2.2, F3.2
- net VUSB: now also C14.1, D26.2 (A), D27.2 (A), D28.1 (K)
- net at D2.1 (K), Q1.2 (G), R3.2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: now also C21.2
- net at BT2.1 (+): now also F2.1; no longer BT1.1 (+)
- net at R17.1: now also U7.6 (GPIO2)
- net at U7.14 (GPIO8): now also R16.2
- net SQPI_SCLK_ESP: no longer names the net of U7.22 (SPICLK)
- net SQPI_SD0_ESP: no longer names the net of U7.24 (SPIQ)
- net SQPI_SD1_ESP: no longer names the net of U7.23 (SPID)
- net SQPI_SD2_ESP: no longer names the net of U7.20 (SPIWP)
- net SQPI_SD3_ESP: no longer names the net of U7.19 (SPIHD)
- net SQPI_SS_ESP: no longer names the net of U7.21 (SPICS0)
- net SQPI_VDD_ESP: no longer names the net of U7.18 (VDD_SPI)
- new net: BT1.1 (+), F3.1
- no-connect marks 6 -> 15
Other:
- note added: "Programmer le courant de charge 2k = 500mA"
- note added: "Static protection"
- note added: "Valider res USB"
- note removed: "5v Reg"
- note removed: "Ajouter une fuse entre les deux cellules?"
- moved on the sheet: BT1, BT2, C1, C16, C17, C18, C19, C20, C22, C23, C24, C25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

Commit message: sleep? no! PCB!
Parts:
- added U4: TP4056, TP4056:TP4056-18650, symbol TP4056:TP4056
Connections:
- net GND: now also U4.2 (GND), U4.4 (Out-), U4.6 (B-)
- net VBATT: now also U4.5 (B+); no longer C2.1, C3.1, L1.1, Q4.3 (S), R26.1, R27.2, R3.1, R6.1, U2.7 (VIN)
- net VUSB: now also U4.1 (5V_IN)
- new net VBAT_LOAD: C2.1, C3.1, L1.1, Q4.3 (S), R26.1, R27.2, R3.1, R6.1, U2.7 (VIN), U4.3 (Out+)
Other:
- moved on the sheet: C1, C14, C4, D3, Q2, R14, R2, R7, R8, TP1, U1

Commit message: Vite! Mon lit m'attend!
Parts:
- removed TP3: USB_P, TestPoint:TestPoint_Loop_D2.54mm_Drill1.5mm_Beaded, symbol Connector:TestPoint
- removed TP5: USB_N, TestPoint:TestPoint_Loop_D2.54mm_Drill1.5mm_Beaded, symbol Connector:TestPoint
Connections:
- net VBATT: no longer JP19.2 (B)
- net VBAT_LOAD: now also JP19.2 (B)
Changed lines of the file:
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@@
 	)
 	(junction
-		(at 469.9 105.41)
-		(diameter 0)
-		(color 0 0 0 0)
-	)
-	(junction
 		(at 156.21 69.85)
 		(diameter 0)
@@
 	)
 	(junction
-		(at 467.36 102.87)
-		(diameter 0)
-		(color 0 0 0 0)
-	)
-	(junction
 		(at 511.81 298.45)
 		(diameter 0)
@@
 	(wire
 		(pts
-			(xy 467.36 102.87) (xy 474.98 102.87)
+			(xy 420.37 102.87) (xy 474.98 102.87)
 		)
 		(stroke
@@
 	(wire
 		(pts
-			(xy 420.37 102.87) (xy 467.36 102.87)
-		)
-		(stroke
-			(width 0)
-			(type default)
-		)
-	)
-	(wire
-		(pts
 			(xy 68.58 300.99) (xy 71.12 300.99)
 		)
@@
 	(wire
 		(pts
-			(xy 420.37 105.41) (xy 469.9 105.41)
-		)
-		(stroke
-			(width 0)
-			(type default)
-		)
-	)
-	(wire
-		(pts
 			(xy 95.25 344.17) (xy 95.25 346.71)
 		)
@@
 	(wire
 		(pts
-			(xy 469.9 105.41) (xy 492.76 105.41)
+			(xy 420.37 105.41) (xy 492.76 105.41)
 		)
 		(stroke
@@
 		)
 	)
-	(label "VBATT"
+	(label "VBAT_LOAD"
 		(at 187.96 262.89 180)
 		(fields_autoplaced yes)
@@
 	)
 	(symbol
-		(lib_id "Connector:TestPoint")
-		(at 467.36 102.87 0)
-		(unit 1)
-		(exclude_from_sim no)
-		(in_bom yes)
-		(on_board yes)
-		(dnp no)
-		(property "Reference" "TP3"
-			(at 467.868 98.298 0)
-			(effects
-				(font
-					(size 1.27 1.27)
-				)
-				(justify left)
-			)
-		)
-		(property "Value" "USB_P"
-			(at 462.915 104.775 0)
-			(effects
-				(font
-					(size 1.27 1.27)
-				)
-				(justify left)
-			)
-		)
-		(property "Footprint" "TestPoint:TestPoint_Loop_D2.54mm_Drill1.5mm_Beaded"
-			(at 472.44 102.87 0)
-			(effects
-				(font
-					(size 1.27 1.27)
-				)
-				(hide yes)
-			)
-		)
-		(property "Datasheet" "~"
-			(at 472.44 102.87 0)
-			(effects
-				(font
-					(size 1.27 1.27)
-				)
-				(hide yes)
-			)
-		)
-		(property "Description" ""
-			(at 467.36 102.87 0)
-			(effects
-				(font
-					(size 1.27 1.27)
-				)
-				(hide yes)
-			)
-		)
-		(pin "1"
-		)
-		(instances
-			(project "SHERPENT20250113"
-				(path "/b9eec091-4b52-44a1-b170-afda02802a46"
-					(reference "TP3")
-					(unit 1)
-				)
-			)
-		)
-	)
-	(symbol
 		(lib_id "LED:WS2812B")
 		(at 450.85 298.45 0)
@@
 					(unit 1)
 				)
-			)
-		)
-	)
-	(symbol
-		(lib_id "Connector:TestPoint")
-		(at 469.9 105.41 0)
-		(unit 1)
-		(exclude_from_sim no)
-		(in_bom yes)
-		(on_board yes)
-		(dnp no)
-		(property "Reference" "TP5"
-			(at 470.408 100.584 0)
-			(effects
-				(font
-					(size 1.27 1.27)
-				)
-				(justify left)
-			)
-		)
-		(property "Value" "USB_N"
-			(at 465.455 107.315 0)
-			(effects
-				(font
-					(size 1.27 1.27)
-				)
-				(justify left)
-			)
-		)
-		(property "Footprint" "TestPoint:TestPoint_Loop_D2.54mm_Drill1.5mm_Beaded"
-			(at 474.98 105.41 0)
-			(effects
-				(font
-					(size 1.27 1.27)
-				)
-				(hide yes)
-			)
-		)
-		(property "Datasheet" "~"
-			(at 474.98 105.41 0)
-			(effects
-				(font
-					(size 1.27 1.27)
-				)
-				(hide yes)
-			)
-		)
-		(property "Description" ""
-			(at 469.9 105.41 0)
-			(effects
-				(font
-					(size 1.27 1.27)
-				)
-				(hide yes)
-			)
-		)
-		(pin "1"
-		)
-		(instances
-			(project "SHERPENT20250113"
-				(path "/b9eec091-4b52-44a1-b170-afda02802a46"
-					(reference "TP5")
-					(unit 1)
-				)
