File: elec/SHERPENT_PCB_RevA/SHERPENT20250113.kicad_sch (KiCad schematic)
At the start: 136 parts, among them J1 2137160001, J2 Conn_01x03_Socket, J3 Conn_01x03_Socket, J4 Conn_01x03_Socket, Q1 NMOS, Q2 PMOS, Q3 NMOS, Q4 PMOS, SW1 CT1102, SW2 SW_Push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

Commit message: ajouté les part numbers dasn revA
Parts:
- C1, C4: DigiKey (none) -> 587-1441-1-ND
- C10, C22, C29, C9: DigiKey (none) -> 587-1248-1-ND
- C11: DigiKey (none) -> 1276-2055-1-ND
- C12: DigiKey (none) -> 490-4771-1-ND
- C14, C17, C21, C24, C3: DigiKey (none) -> 311-1344-1-ND
- C15, C2: DigiKey (none) -> 587-1256-1-ND
- C16, C18: DigiKey (none) -> 490-6215-1-ND
- C19, C26: DigiKey (none) -> 490-4781-1-ND
- C20: DigiKey (none) -> 1276-1450-1-ND
- C23: DigiKey (none) -> 311-3566-1-ND
- C25: DigiKey (none) -> 490-10024-1-ND
- C27, C28: DigiKey (none) -> 490-8080-1-ND
- C5: value 100nf -> 100n; DigiKey (none) -> 311-1344-1-ND
- C6: DigiKey (none) -> 490-4520-1-ND
- C7, C8: DigiKey (none) -> 732-8793-1-ND
- D1, D2, D25: DigiKey (none) -> TSS54URGGCT-ND
- D6: now not fitted
- F2, F3: DigiKey (none) -> 5923-0686F8000-01CT-ND
- J1: DigiKey (none) -> 2073-USB4085-GF-ACT-ND
- L2: DigiKey (none) -> 490-1078-1-ND
- L3: DigiKey (none) -> 490-15076-1-ND
- Q1, Q3: DigiKey (none) -> 448-SN7002NH6433XTMA1CT-ND
- Q2, Q4: DigiKey (none) -> BSS84PH6327XTSA2CT-ND
- R1, R10, R16, R17, R20, R22, R25, R3, R4, R5, R6, R9: DigiKey (none) -> 311-5.10KHRCT-ND
- R11: DigiKey (none) -> 311-45.3KHRCT-ND
- R12: DigiKey (none) -> 311-357KHRCT-ND
- R13: DigiKey (none) -> 311-48.7KHRCT-ND
- R14, R2, R28: DigiKey (none) -> P100KHCT-ND
- R18, R21, R26: DigiKey (none) -> 311-0.0GRCT-ND
- R23: DigiKey (none) -> 311-130HRCT-ND; now not fitted
- R24: DigiKey (none) -> P0.0JCT-ND
- R7: DigiKey (none) -> 311-470GRCT-ND
- R8: DigiKey (none) -> P2.00KHCT-ND
- SW1: DigiKey (none) -> 2449-CT1102V3.15F100-ND
- SW2: DigiKey (none) -> 2449-CS1213AGF260CT-ND
- U2: DigiKey (none) -> 296-TPS61288LRQQRCT-ND
- U5: DigiKey (none) -> 497-1241-1-ND
- U7: DigiKey (none) -> 1904-ESP32-C3FH4CT-ND
- Y1: DigiKey (none) -> 535-15013-1-ND
